File: payload_board.kicad_sch (KiCad schematic)
At the start: 92 parts, among them IC1 RP2040_QFN56, IC2 AZ1117CH-3.3TRG1, J1 Cam_PicoLock, J10 503398-1892, J11 Stemma, J15 Debug_Conn, J2 Cam_Conn, J3 Antenna_Conn, J4 usb jumper, J5 Display_Conn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

Commit message: Updated for v1.0 manufacturing
Parts:
- removed R9: 10k, Connector_PinSocket_2.54mm:PinSocket_1x02_P2.54mm_Vertical, symbol Device:R_US
- added JP2: SolderJumper_2_Open, Jumper:SolderJumper-2_P1.3mm_Open_RoundedPad1.0x1.5mm, symbol Jumper:SolderJumper_2_Open
Connections:
- net ~{RESET}: now also JP2.2 (B)
- net at U2.7 (~{RESET}): now also JP2.1 (A)
Other:
- note removed: "WDT enabled when installed"
Changed lines of the file:
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@@
 		)
 	)
-	(polyline
-		(pts
-			(xy 184.15 123.19) (xy 201.93 123.19)
-		)
-		(stroke
-			(width 0)
-			(type default)
-		)
-	)
 	(wire
 		(pts
@@
 		)
 	)
-	(polyline
-		(pts
-			(xy 184.15 130.81) (xy 184.15 123.19)
-		)
-		(stroke
-			(width 0)
-			(type default)
-		)
-	)
 	(wire
 		(pts
@@
 		)
 	)
-	(polyline
-		(pts
-			(xy 201.93 130.81) (xy 184.15 130.81)
-		)
-		(stroke
-			(width 0)
-			(type default)
-		)
-	)
 	(wire
 		(pts
@@
 		)
 	)
-	(polyline
-		(pts
-			(xy 201.93 123.19) (xy 201.93 130.81)
-		)
-		(stroke
-			(width 0)
-			(type default)
-		)
-	)
 	(wire
 		(pts
@@
 		)
 	)
-	(text "WDT enabled\nwhen installed"
-		(exclude_from_sim no)
-		(at 191.77 128.27 0)
-		(effects
-			(font
-				(size 0.889 0.889)
-			)
-			(justify left bottom)
-		)
-	)
 	(text "Camera Shunt"
 		(exclude_from_sim no)
@@
 		)
 	)
-	(global_label "GND"
-		(shape bidirectional)
-		(at 238.76 120.65 0)
-		(fields_autoplaced yes)
-		(effects
-			(font
-				(size 0.254 0.254)
-			)
-			(justify left)
-		)
-		(property "Intersheetrefs" "${INTERSHEET_REFS}"
-			(at 138.43 72.39 0)
-			(effects
-				(font
-					(size 1.27 1.27)
-				)
-				(hide yes)
-			)
-		)
-	)
 	(global_label "SPI0_MISO"
 		(shape input)
@@
 		)
 	)
-	(global_label "GND"
-		(shape bidirectional)
-		(at 203.2 125.73 0)
-		(fields_autoplaced yes)
-		(effects
-			(font
-				(size 0.254 0.254)
-			)
-			(justify left)
-		)
-		(property "Intersheetrefs" "${INTERSHEET_REFS}"
-			(at 138.43 72.39 0)
-			(effects
-				(font
-					(size 1.27 1.27)
-				)
-				(hide yes)
-			)
-		)
-	)
 	(global_label "DIN-"
 		(shape input)
@@
 	)
 	(symbol
-		(lib_id "Device:R_US")
-		(at 190.5 127 0)
-		(mirror x)
-		(unit 1)
-		(exclude_from_sim no)
-		(in_bom yes)
-		(on_board yes)
-		(dnp no)
-		(property "Reference" "R9"
-			(at 186.69 125.73 0)
-			(effects
-				(font
-					(size 1.27 1.27)
-				)
-			)
-		)
-		(property "Value" "10k"
-			(at 186.69 128.27 0)
-			(effects
-				(font
-					(size 1.27 1.27)
-				)
-			)
-		)
-		(property "Footprint" "Connector_PinSocket_2.54mm:PinSocket_1x02_P2.54mm_Vertical"
-			(at 191.516 126.746 90)
-			(effects
-				(font
-					(size 1.27 1.27)
-				)
-				(hide yes)
-			)
-		)
-		(property "Datasheet" "~"
-			(at 190.5 127 0)
-			(effects
-				(font
-					(size 1.27 1.27)
-				)
-				(hide yes)
-			)
-		)
-		(property "Description" "10k 0603"
-			(at 186.69 128.27 0)
-			(effects
-				(font
-					(size 1.27 1.27)
-				)
-				(hide yes)
-			)
-		)
-		(property "DNI" "DNI"
-			(at 195.58 129.54 0)
-			(effects
-				(font
-					(size 1.27 1.27)
-					(bold yes)
-				)
-			)
-		)
-		(pin "1"
-		)
-		(pin "2"
-		)
-		(instances
-			(project "payload_board"
-				(path "/e3f40ef2-c677-4aae-b100-4b87fee46bc8"
-					(reference "R9")
-					(unit 1)
-				)
-			)
-			(project "FC_Board_v1"
-				(path "/e63e39d7-6ac0-4ffd-8aa3-1841a4541b55"
-					(reference "R2")
-					(unit 1)
-				)
-			)
-		)
-	)
-	(symbol
 		(lib_id "Device:C")
 		(at 289.56 143.51 90)
@@
 					(unit 1)
 				)
+			)
+		)
+	)
+	(symbol
+		(lib_name "SolderJumper_2_Open_1")
+		(lib_id "Jumper:SolderJumper_2_Open")
+		(at 190.5 127 270)
+		(unit 1)
+		(exclude_from_sim yes)
+		(in_bom no)
+		(on_board yes)
+		(dnp no)
+		(property "Reference" "JP2"
+			(at 193.04 125.7299 90)
+			(effects
+				(font
+					(size 1.27 1.27)
+				)
+				(justify left)
+			)
+		)
+		(property "Value" "SolderJumper_2_Open"
+			(at 180.086 130.048 90)
+			(effects
+				(font
+					(size 1.27 1.27)
+				)
+				(justify left)
+			)
+		)
+		(property "Footprint" "Jumper:SolderJumper-2_P1.3mm_Open_RoundedPad1.0x1.5mm"
+			(at 190.5 127 0)
+			(effects
+				(font
+					(size 1.27 1.27)
+				)
+				(hide yes)
+			)
+		)
+		(property "Datasheet" "~"
+			(at 190.5 127 0)
+			(effects
+				(font
+					(size 1.27 1.27)
+				)
+				(hide yes)
+			)
+		)
+		(property "Description" "Solder Jumper, 2-pole, open"
+			(at 190.5 127 0)
+			(effects
+				(font
+					(size 1.27 1.27)
+				)
+				(hide yes)
+			)
+		)
+		(pin "2"
+		)
+		(pin "1"
+		)
+		(instances
+			(project ""
+				(path "/e3f40ef2-c677-4aae-b100-4b87fee46bc8"
+					(reference "JP2")
+					(unit 1)
+				)

Commit message: added meme
Parts:
- C18: footprint Capacitor_SMD:C_1206_3216Metric_Pad1.33x1.80mm_HandSolder -> Capacitor_SMD:C_0603_1608Metric_Pad1.08x0.95mm_HandSolder
- J1: footprint PayloadBoard:Molex_Pico_CON_5040500891 -> PayloadBoard:Molex_Pico_CON_5040500691
Changed lines of the file:
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@@
 	(label "~{RESET}"
 		(at 190.5 135.89 0)
-		(fields_autoplaced yes)
 		(effects
 			(font
@@
 	(label "QSPI_CS"
 		(at 198.8092 80.0257 0)
-		(fields_autoplaced yes)
 		(effects
 			(font
@@
 	(label "D+"
 		(at 140.97 177.8 0)
-		(fields_autoplaced yes)
 		(effects
 			(font
@@
 	(label "USBBOOT"
 		(at 130.81 95.25 0)
-		(fields_autoplaced yes)
 		(effects
 			(font
@@
 	(label "QSPI_SCK"
 		(at 36.83 123.19 0)
-		(fields_autoplaced yes)
 		(effects
 			(font
@@
 	(label "SWDIO"
 		(at 135.89 140.97 0)
-		(fields_autoplaced yes)
 		(effects
 			(font
@@
 	(label "QSPI_SCK"
 		(at 196.2692 72.4057 0)
-		(fields_autoplaced yes)
 		(effects
 			(font
@@
 	(label "QSPI_DATA[1]"
 		(at 196.2692 77.4857 0)
-		(fields_autoplaced yes)
 		(effects
 			(font
@@
 	(label "USBBOOT"
 		(at 153.67 212.09 180)
-		(fields_autoplaced yes)
 		(effects
 			(font
@@
 	(label "QSPI_DATA[3]"
 		(at 196.2692 85.1057 0)
-		(fields_autoplaced yes)
 		(effects
 			(font
@@
 	(label "D-"
 		(at 147.32 130.81 0)
-		(fields_autoplaced yes)
 		(effects
 			(font
@@
 	(label "QSPI_DATA[2]"
 		(at 36.83 133.35 0)
-		(fields_autoplaced yes)
 		(effects
 			(font
@@
 	(label "VCC"
 		(at 196.85 210.82 0)
-		(fields_autoplaced yes)
 		(effects
 			(font
@@
 	(label "SWCLK"
 		(at 135.89 138.43 0)
-		(fields_autoplaced yes)
 		(effects
 			(font
@@
 	(label "QSPI_DATA[0]"
 		(at 196.2692 74.9457 0)
-		(fields_autoplaced yes)
 		(effects
 			(font
@@
 	(label "QSPI_CS"
 		(at 36.83 125.73 0)
-		(fields_autoplaced yes)
 		(effects
 			(font
@@
 	(label "QSPI_DATA[1]"
 		(at 36.83 130.81 0)
-		(fields_autoplaced yes)
 		(effects
 			(font
@@
 	(label "3Vo"
 		(at 26.67 231.14 0)
-		(fields_autoplaced yes)
 		(effects
 			(font
@@
 	(label "D+"
 		(at 147.32 133.35 0)
-		(fields_autoplaced yes)
 		(effects
 			(font
@@
 	(label "QSPI_CS"
 		(at 132.08 219.71 270)
-		(fields_autoplaced yes)
 		(effects
 			(font
@@
 	(label "IMURX"
 		(at 204.47 205.74 0)
-		(fields_autoplaced yes)
 		(effects
 			(font
@@
 	(label "D-"
 		(at 140.97 175.26 0)
-		(fields_autoplaced yes)
 		(effects
 			(font
@@
 	(label "QSPI_DATA[0]"
 		(at 36.83 128.27 0)
-		(fields_autoplaced yes)
 		(effects
 			(font
@@
 	(label "QSPI_DATA[2]"
 		(at 196.2692 82.5657 0)
-		(fields_autoplaced yes)
 		(effects
 			(font
@@
 	(label "QSPI_DATA[3]"
 		(at 36.83 135.89 0)
-		(fields_autoplaced yes)
 		(effects
 			(font
@@
 	(label "IMUTX"
 		(at 207.01 208.28 0)
-		(fields_autoplaced yes)
 		(effects
 			(font
@@
 	(label "~{RESET}"
 		(at 39.37 62.23 0)
-		(fields_autoplaced yes)
 		(effects
 			(font
@@
 			)
 		)
-		(property "Footprint" "Capacitor_SMD:C_1206_3216Metric_Pad1.33x1.80mm_HandSolder"
+		(property "Footprint" "Capacitor_SMD:C_0603_1608Metric_Pad1.08x0.95mm_HandSolder"
 			(at 371.8052 25.4 0)
 			(effects
@@
 			)
 		)
-		(property "Footprint" "PayloadBoard:Molex_Pico_CON_5040500891"
+		(property "Footprint" "PayloadBoard:Molex_Pico_CON_5040500691"
 			(at 25.4 176.53 0)
 			(effects
